Commit message: 3.25

File: src/fishbot_description/urdf/fishbot/fishbot.ros2_control.xacro (robot description, xacro)
@@ -1,5 +1,5 @@
 <?xml version="1.0"?>
 <robot xmlns:xacro="http://www.ros.org/wiki/xacro">
-    <xacro:macro name="fishbot_ros2_control">
+    <xacro:macro name="fishbot_ros2_control" params="controller_config:='$(find fishbot_description)/config/fishbot_ros2_controller.yaml'">
     <ros2_control name="FishBotGazeboSystem" type="system">
             <hardware>
@@ -35,5 +35,5 @@
         <gazebo>
         <plugin filename="libgazebo_ros2_control.so" name="gazebo_ros2_control">
-            <parameters>$(find fishbot_description)/config/fishbot_ros2_controller.yaml</parameters>
+            <parameters>${controller_config}</parameters>
             <ros>
                 <remapping>/fishbot_diff_drive_controller/cmd_vel_unstamped:=/cmd_vel</remapping>

File: src/fishbot_description/urdf/fishbot/fishbot.urdf.xacro (robot description, xacro)
@@ -1,27 +1,23 @@
 <?xml version="1.0"?>
 <robot xmlns:xacro="http://www.ros.org/wiki/xacro" name="fishbot">
+    <xacro:arg name="controller_config" default="$(find fishbot_description)/config/fishbot_ros2_controller.yaml" />
     <xacro:include filename="$(find fishbot_description)/urdf/fishbot/base.urdf.xacro" />
-    <!-- 传感器组件 -->
     <xacro:include filename="$(find fishbot_description)/urdf/fishbot/sensor/imu.urdf.xacro" />
     <xacro:include filename="$(find fishbot_description)/urdf/fishbot/sensor/laser.urdf.xacro" />
     <xacro:include filename="$(find fishbot_description)/urdf/fishbot/sensor/camera.urdf.xacro" />
-     <!-- 执行器组件 -->
     <xacro:include filename="$(find fishbot_description)/urdf/fishbot/actuator/wheel.urdf.xacro" />
     <xacro:include filename="$(find fishbot_description)/urdf/fishbot/actuator/caster.urdf.xacro" />
     <xacro:base_xacro length="0.12" radius="0.1" />
-    <!-- 传感器 -->
     <xacro:imu_xacro xyz="0 0 0.02" />
     <xacro:laser_xacro xyz="0 0 0.10" />
     <xacro:camera_xacro xyz="0.10 0 0.075" />
-    <!-- 执行器主动轮+从动轮 -->
     <xacro:wheel_xacro wheel_name="left" xyz="0 0.10 -0.06" />
     <xacro:wheel_xacro wheel_name="right" xyz="0 -0.10 -0.06" />
     <xacro:caster_xacro caster_name="front" xyz="0.08 0.0 -0.076" />
     <xacro:caster_xacro caster_name="back" xyz="-0.08 0.0 -0.076" />
-    <!-- Gazebo 插件 -->
     <xacro:include filename="$(find fishbot_description)/urdf/fishbot/plugins/gazebo_control_plugin.xacro" />
     <!-- <xacro:gazebo_control_plugin /> -->
     <xacro:include filename="$(find fishbot_description)/urdf/fishbot/fishbot.ros2_control.xacro" />
-    <xacro:fishbot_ros2_control />
+    <xacro:fishbot_ros2_control controller_config="$(arg controller_config)" />
     <xacro:include filename="$(find fishbot_description)/urdf/fishbot/plugins/gazebo_sensor_plugin.xacro" />
     <xacro:gazebo_sensor_plugin />
